File: _saved_bq25071 Breakout.sch (KiCad schematic (older format))
At the start: 19 parts, among them P1 USB_OTG, P2 CONN_01X05, P3 CONN_01X04, P4 CONN_01X02, U1 bq25071

Commit message: pcb layout
Parts:
- P1: footprint (none) -> connectors:USB_MICRO_B_MOLEX
Changed lines of the file:
@@
 LIBS:valves
 LIBS:bq25071
+LIBS:bq25071 Breakout-cache
 EELAYER 25 0
 EELAYER END
@@
 F 0 "P1" H 5175 4175 50  0000 C CNN
 F 1 "USB_OTG" H 4850 4500 50  0000 C CNN
-F 2 "" V 4800 4200 50  0001 C CNN
+F 2 "connectors:USB_MICRO_B_MOLEX" V 4800 4200 50  0001 C CNN
 F 3 "" V 4800 4200 50  0000 C CNN
 	1    4850 4300
