File: bq25071 Breakout.sch (KiCad schematic (older format))
At the start: 19 parts, among them P1 USB_OTG, P2 CONN_01X05, P3 CONN_01X04, P4 CONN_01X02, U1 bq25071

Commit message: better component placement
Parts:
- F1: footprint Resistors_SMD:R_1812 -> Resistors_SMD:R_1206
Changed lines of the file:
@@
 F 0 "F1" V 4350 4700 50  0000 C CNN
 F 1 "500mA" V 4550 4700 50  0000 C CNN
-F 2 "Resistors_SMD:R_1812" H 4500 4500 50  0001 L CNN
+F 2 "Resistors_SMD:R_1206" H 4500 4500 50  0001 L CNN
 F 3 "" H 4450 4700 50  0001 C CNN
 	1    4450 4700

Commit message: change battery connector to jst xh (seems to be standard for rc lipos)
Parts:
- P4: footprint Connectors_JST:JST_PH_S2B-PH-SM4-TB_02x2.00mm_Angled -> Connectors_JST:JST_XH_B02B-XH-A_02x2.50mm_Straight
Changed lines of the file:
@@
 F 0 "P4" H 7750 4550 50  0000 C CNN
 F 1 "CONN_01X02" V 7850 4400 50  0000 C CNN
-F 2 "Connectors_JST:JST_PH_S2B-PH-SM4-TB_02x2.00mm_Angled" H 7750 4400 50  0001 C CNN
+F 2 "Connectors_JST:JST_XH_B02B-XH-A_02x2.50mm_Straight" H 7750 4400 50  0001 C CNN
 F 3 "" H 7750 4400 50  0000 C CNN
 	1    7750 4400
